File: io_module/io_module.kicad_sch (KiCad schematic)
At the start: 9 parts, among them J1 8P, J2 10P, J3 8P, J4 10P, J5 EA, J6 EB, U1 MCP23S17_ML

Commit message: io expansion board r2
Connections:
- net PB2: now also R1.1, U1.7 (~{CS})
- net PC3: no longer R1.1, U1.7 (~{CS})
Changed lines of the file:
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@@
     (stroke (width 0) (type default) (color 0 0 0 0))
   )
-  (wire (pts (xy 43.18 45.72) (xy 63.5 45.72))
+  (wire (pts (xy 43.18 45.72) (xy 50.8 45.72))
     (stroke (width 0) (type default) (color 0 0 0 0))
   )
@@
     (stroke (width 0) (type default) (color 0 0 0 0))
   )
+  (wire (pts (xy 43.18 43.18) (xy 63.5 43.18))
+    (stroke (width 0) (type default) (color 0 0 0 0))
+  )
   (wire (pts (xy 71.12 30.48) (xy 71.12 27.94))
     (stroke (width 0) (type default) (color 0 0 0 0))
@@
     (stroke (width 0) (type default) (color 0 0 0 0))
   )
-  (wire (pts (xy 43.18 43.18) (xy 63.5 43.18))
-    (stroke (width 0) (type default) (color 0 0 0 0))
-  )
   (wire (pts (xy 170.18 60.96) (xy 179.07 60.96))
     (stroke (width 0) (type default) (color 0 0 0 0))
@@
     (effects (font (size 1.27 1.27)) (justify right bottom))
   )
-  (label "~{RESET}" (at 63.5 43.18 180)
-    (effects (font (size 1.27 1.27)) (justify right bottom))
-  )
   (label "PC3" (at 76.2 45.72 0)
     (effects (font (size 1.27 1.27)) (justify left bottom))
@@
     (effects (font (size 1.27 1.27)) (justify right bottom))
   )
-  (label "~{CS}" (at 63.5 45.72 180)
-    (effects (font (size 1.27 1.27)) (justify right bottom))
-  )
+  (label "~{CS}" (at 63.5 43.18 180)
+    (effects (font (size 1.27 1.27)) (justify right bottom))
+  )
